Commit message: fix: balance friction and stiffness parameters to resolve Gazebo solver gridlock

File: urdf/atm_gazebo.xacro (robot description, xacro)
@@ -2,30 +2,48 @@
 <robot name="atm" xmlns:xacro="http://ros.org/wiki/xacro">
     <gazebo reference="wheel_left_link">
-        <mu1>10000000000.0</mu1>
-        <mu2>10000000000.0</mu2>
-        <kp>10000000000.0</kp>
+        <mu1>2.0</mu1> <mu2>2.0</mu2>
+        <kp>1000000.0</kp> <kd>10.0</kd>
+        <minDepth>0.001</minDepth>
+        <material>Gazebo/Black</material>
+    </gazebo>
+    <gazebo reference="wheel_right_link">
+        <mu1>2.0</mu1>
+        <mu2>2.0</mu2>
+        <kp>1000000.0</kp>
         <kd>10.0</kd>
         <minDepth>0.001</minDepth>
-    </gazebo>
-    <gazebo reference="wheel_right_link">
-        <mu1>10000000000.0</mu1>
-        <mu2>10000000000.0</mu2>
-        <kp>10000000000.0</kp>
-        <kd>10.0</kd>
-        <minDepth>0.001</minDepth>
+        <material>Gazebo/Black</material>
     </gazebo>
     <gazebo reference="caster_front_link">
-        <mu1>0.1</mu1>
-        <mu2>0.1</mu2>
-        <kp>1000000000.0</kp>
+        <mu1>0.0</mu1>
+        <mu2>0.0</mu2>
+        <kp>1000000.0</kp>
         <kd>100.0</kd>
         <minDepth>0.001</minDepth>
+        <material>Gazebo/White</material>
     </gazebo>
     <gazebo reference="caster_rear_link">
-        <mu1>0.1</mu1>
-        <mu2>0.1</mu2>
-        <kp>1000000000.0</kp>
+        <mu1>0.0</mu1>
+        <mu2>0.0</mu2>
+        <kp>1000000.0</kp>
         <kd>100.0</kd>
         <minDepth>0.001</minDepth>
+        <material>Gazebo/White</material>
+    </gazebo>
+    <gazebo>
+        <plugin name="diff_drive" filename="libgazebo_ros_diff_drive.so">
+            <update_rate>30</update_rate>
+            <left_joint>wheel_left_joint</left_joint>
+            <right_joint>wheel_right_joint</right_joint>
+            <wheel_separation>0.1402</wheel_separation>
+            <wheel_diameter>0.066</wheel_diameter>
+            <max_wheel_torque>20</max_wheel_torque>
+            <max_wheel_acceleration>1.0</max_wheel_acceleration>
+            <publish_odom>true</publish_odom>
+            <publish_odom_tf>true</publish_odom_tf>
+            <publish_wheel_tf>true</publish_wheel_tf>
+            <odometry_frame>odom</odometry_frame>
+            <robot_base_frame>base_footprint</robot_base_frame>
+        </plugin>
     </gazebo>
 </robot>
